Commit message: v3.6添加预编译编译aarch64版

File: model/AzureLoong.urdf (robot description, URDF)
Before this commit: robot OpenLoog, 32 links, 31 joints
Links:
- link Link_ankle_l_pitch: geometry collision mesh filename=meshes/Link_ankle_l_pitch.STL; visual mesh filename=meshes/Link_ankle_l_pitch.STL
- link Link_ankle_l_roll: geometry collision mesh filename=meshes/Link_ankle_l_roll.STL; visual mesh filename=meshes/Link_ankle_l_roll.STL
- link Link_ankle_r_pitch: geometry collision mesh filename=meshes/Link_ankle_r_pitch.STL; visual mesh filename=meshes/Link_ankle_r_pitch.STL
- link Link_ankle_r_roll: geometry collision mesh filename=meshes/Link_ankle_r_roll.STL; visual mesh filename=meshes/Link_ankle_r_roll.STL
- link Link_arm_l_01: mass 0.756406339732892 -> 0.999469576; geometry collision mesh filename=meshes/Link_arm_l_01.STL; visual mesh filename=meshes/Link_arm_l_01.STL
- link Link_arm_l_02: mass 0.984999996273518 -> 1.2000362; geometry collision mesh filename=meshes/Link_arm_l_02.STL; visual mesh filename=meshes/Link_arm_l_02.STL
- link Link_arm_l_03: mass 0.958999855228925 -> 1.05028474; geometry collision mesh filename=meshes/Link_arm_l_03.STL; visual mesh filename=meshes/Link_arm_l_03.STL
- link Link_arm_l_04: mass 0.60000012303258 -> 0.80390762; geometry collision mesh filename=meshes/Link_arm_l_04.STL; visual mesh filename=meshes/Link_arm_l_04.STL
- link Link_arm_l_05: mass 0.68976 -> 0.80390762; geometry collision mesh filename=meshes/Link_arm_l_05.STL; visual mesh filename=meshes/Link_arm_l_05.STL
- link Link_arm_l_06: mass 0.280000012776158 -> 0.466149172; geometry collision mesh filename=meshes/Link_arm_l_06.STL; visual mesh filename=meshes/Link_arm_l_06.STL
- link Link_arm_l_07: mass 0.61354 -> 0.6529339; geometry collision mesh filename=meshes/Link_arm_l_07.STL; visual mesh filename=meshes/Link_arm_l_07.STL
- link Link_arm_r_01: mass 0.75641 -> 1.0002100; geometry collision mesh filename=meshes/Link_arm_r_01.STL; visual mesh filename=meshes/Link_arm_r_01.STL
- link Link_arm_r_02: mass 0.984999996273518 -> 1.19958456; geometry collision mesh filename=meshes/Link_arm_r_02.STL; visual mesh filename=meshes/Link_arm_r_02.STL
- link Link_arm_r_03: mass 0.958999855228924 -> 1.0507333; geometry collision mesh filename=meshes/Link_arm_r_03.STL; visual mesh filename=meshes/Link_arm_r_03.STL
- link Link_arm_r_04: mass 0.6 -> 0.688970829; geometry collision mesh filename=meshes/Link_arm_r_04.STL; visual mesh filename=meshes/Link_arm_r_04.STL
- link Link_arm_r_05: mass 0.68976 -> 0.80390762; geometry collision mesh filename=meshes/Link_arm_r_05.STL; visual mesh filename=meshes/Link_arm_r_05.STL
- link Link_arm_r_06: mass 0.28 -> 0.466149172; geometry collision mesh filename=meshes/Link_arm_r_06.STL; visual mesh filename=meshes/Link_arm_r_06.STL
- link Link_arm_r_07: mass 0.61354 -> 0.6529339; geometry collision mesh filename=meshes/Link_arm_r_07.STL; visual mesh filename=meshes/Link_arm_r_07.STL
- link Link_head_pitch: mass 1.3943 -> 2.65751; geometry collision mesh filename=meshes/Link_head_pitch.STL; visual mesh filename=meshes/Link_head_pitch.STL
- link Link_head_yaw: geometry collision mesh filename=meshes/Link_head_yaw.STL; visual mesh filename=meshes/Link_head_yaw.STL
- link Link_hip_l_pitch: geometry collision mesh filename=meshes/Link_hip_l_pitch.STL; visual mesh filename=meshes/Link_hip_l_pitch.STL
- link Link_hip_l_roll: geometry collision mesh filename=meshes/Link_hip_l_roll.STL; visual mesh filename=meshes/Link_hip_l_roll.STL
- link Link_hip_l_yaw: geometry collision mesh filename=meshes/Link_hip_l_yaw.STL; visual mesh filename=meshes/Link_hip_l_yaw.STL
- link Link_hip_r_pitch: geometry collision mesh filename=meshes/Link_hip_r_pitch.STL; visual mesh filename=meshes/Link_hip_r_pitch.STL
- link Link_hip_r_roll: geometry collision mesh filename=meshes/Link_hip_r_roll.STL; visual mesh filename=meshes/Link_hip_r_roll.STL
- link Link_hip_r_yaw: geometry collision mesh filename=meshes/Link_hip_r_yaw.STL; visual mesh filename=meshes/Link_hip_r_yaw.STL
- link Link_knee_l_pitch: geometry collision mesh filename=meshes/Link_knee_l_pitch.STL; visual mesh filename=meshes/Link_knee_l_pitch.STL
- link Link_knee_r_pitch: geometry collision mesh filename=meshes/Link_knee_r_pitch.STL; visual mesh filename=meshes/Link_knee_r_pitch.STL
- link Link_waist_pitch: mass 2.6964 -> 3.1347677; geometry collision mesh filename=meshes/Link_waist_pitch.STL; visual mesh filename=meshes/Link_waist_pitch.STL
- link Link_waist_roll: mass 2.9806 -> 3.2000000; geometry collision mesh filename=meshes/Link_waist_roll.STL; visual mesh filename=meshes/Link_waist_roll.STL
- link Link_waist_yaw: mass 7.3588 -> 7.6000000; geometry collision mesh filename=meshes/Link_waist_yaw.STL; visual mesh filename=meshes/Link_waist_yaw.STL
- link base_link: mass 22.447 -> 27.0000000; geometry collision mesh filename=meshes/base_link.STL; visual mesh filename=meshes/base_link.STL
Joints:
- joint J_arm_l_01: origin xyz=0.004 0.1616 0.3922 rpy=0 0 0 -> xyz=0 0.15585 0.4005 rpy=0 0 0
- joint J_arm_l_02: limit lower=-1.83260 upper=1.83260 effort=80 velocity=3.14 -> lower=-1.832595715 upper=1.832595715 effort=80 velocity=3.14; origin xyz=0.042 0.041 0 rpy=0 0 0 -> xyz=0 0.062 0 rpy=0 0 0
- joint J_arm_l_03: limit lower=-2.96706 upper=2.96706 effort=48 velocity=3.14 -> lower=-2.967059728 upper=2.967059728 effort=58 velocity=3.14; origin xyz=-0.042 0.1226 0 rpy=0 0 0 -> xyz=0 0.1226 -4.5237E-05 rpy=0 0 0
- joint J_arm_l_04: limit lower=0 upper=2.96706 effort=48 velocity=3.14 -> lower=0 upper=2.967059728 effort=58 velocity=3.14; origin xyz=-0.0353 0.1774 0.024 rpy=0 0 0 -> xyz=0 0.1774 0.024 rpy=0 0 0
- joint J_arm_l_05: limit lower=-2.96706 upper=2.96706 effort=12.4 velocity=6.28 -> lower=-2.967059728 upper=2.967059728 effort=11.5 velocity=6.28; origin xyz=0.0353 0.1035 -0.024 rpy=0 0 0 -> xyz=0 0.107 -0.024 rpy=0 0 0
- joint J_arm_l_06: limit lower=-1.8326 upper=1.8326 effort=12.4 velocity=6.28 -> lower=-1.570796327 upper=1.570796327 effort=11.5 velocity=6.28; origin xyz=0.0265 0.1965 0 rpy=0 0 0 -> xyz=0 0.139 0 rpy=0 0 0
- joint J_arm_l_07: limit lower=-1.04720 upper=1.04720 effort=12.4 velocity=6.28 -> lower=-1.308996939 upper=1.308996939 effort=11.5 velocity=6.28; origin xyz=-0.0265 0 0.0318 rpy=0 0 0 -> xyz=0 0.054 4.52E-05 rpy=0 0 0
- joint J_arm_r_01: origin xyz=0.004 -0.1616 0.3922 rpy=0 0 0 -> xyz=0 -0.15585 0.4005 rpy=0 0 0
- joint J_arm_r_02: limit lower=-1.83260 upper=1.83260 effort=80 velocity=3.14 -> lower=-1.8326 upper=1.8326 effort=80 velocity=3.14; origin xyz=-0.042 -0.041 0 rpy=0 0 0 -> xyz=0 -0.062 0 rpy=0 0 0
- joint J_arm_r_03: limit lower=-2.96706 upper=2.96706 effort=48 velocity=3.14 -> lower=-2.967059728 upper=2.967059728 effort=58 velocity=3.14; origin xyz=0.042 -0.1226 0 rpy=0 0 0 -> xyz=0 -0.1226 -4.5237E-05 rpy=0 0 0
- joint J_arm_r_04: limit lower=0 upper=2.96706 effort=48 velocity=3.14 -> lower=0 upper=2.967059728 effort=58 velocity=3.14; origin xyz=0.0353 -0.1774 0.024 rpy=0 0 0 -> xyz=0 -0.1774 0.024045 rpy=0 0 0
- joint J_arm_r_05: axis 0 1 0 -> 0 -1 0; limit lower=-2.96706 upper=2.96706 effort=12.4 velocity=6.28 -> lower=-2.967059728 upper=2.967059728 effort=11.5 velocity=6.28; origin xyz=-0.0353 -0.1035 -0.024 rpy=0 0 0 -> xyz=0 -0.107 -0.024045 rpy=0 0 0
- joint J_arm_r_06: limit lower=-1.8326 upper=1.8326 effort=12.4 velocity=6.28 -> lower=-1.570796327 upper=1.570796327 effort=11.5 velocity=6.28; origin xyz=-0.0265 -0.1965 0 rpy=0 0 0 -> xyz=0 -0.139 4.5237E-05 rpy=0 0 0
- joint J_arm_r_07: limit lower=-1.04720 upper=1.04720 effort=12.4 velocity=6.28 -> lower=-1.308996939 upper=1.308996939 effort=11.5 velocity=6.28; origin xyz=0.0265 0 0.0318 rpy=0 0 0 -> xyz=0 -0.054 0 rpy=0 0 0
